Commit message: Added more simulation

File: sim/inmoov/inmoov.urdf.xacro (robot description, xacro)
@@ -1,112 +1,284 @@
 <?xml version="1.0"?>
-<robot name="inmoov" xmlns:xacro="http://ros.org/wiki/xacro">
-<xacro:include filename="$(find inmoov_description)/urdf/config.joints.urdf.xacro" />
-<xacro:include filename="$(find inmoov_description)/urdf/config.inertial.urdf.xacro" />
-<xacro:include filename="$(find inmoov_description)/urdf/materials.urdf.xacro" />
-<xacro:include filename="$(find inmoov_description)/urdf/inmoov.gazebo" />
-  <xacro:include filename="$(find inmoov_description)/urdf/materials.urdf.xacro" />
-  <xacro:include filename="$(find inmoov_description)/urdf/asmBase.urdf.xacro" />
-  <xacro:include filename="$(find inmoov_description)/urdf/asmTorso.urdf.xacro" />
-  <xacro:include filename="$(find inmoov_description)/urdf/asmHead.urdf.xacro" />
-  <xacro:include filename="$(find inmoov_description)/urdf/asmEye.urdf.xacro" />
-  <xacro:include filename="$(find inmoov_description)/urdf/asmFace.urdf.xacro" />
-  <xacro:include filename="$(find inmoov_description)/urdf/asmArm.urdf.xacro" />
-  <xacro:include filename="$(find inmoov_description)/urdf/asmHand.urdf.xacro" />
+<!--
+This file was originally a ROS xacro. PyBullet does not process xacro macros/includes.
+To make it usable in PyBullet, it has been converted into plain URDF (no xacro tags,
+no ROS $(find ...) includes, and no package:// mesh URLs).
+Mesh paths are relative to this directory: `meshes/...`
+-->
+<robot name="inmoov">
+  <!-- Simple materials (optional in PyBullet, but keeps visuals valid URDF). -->
+  <material name="base_gray"><color rgba="0.75 0.75 0.75 1"/></material>
+  <material name="frame_green"><color rgba="0.2 0.9 0.2 1"/></material>
   <link name="world"/>
   <joint name="fixed" type="fixed">
     <parent link="world"/>
     <child link="base_link"/>
+    <origin rpy="0 0 0" xyz="0 0 0"/>
   </joint>
   <link name="base_link">
-    <visual>
-      <geometry>
-        <cylinder length="0.11" radius="0.26"/>
-      </geometry>
+    <inertial>
       <origin rpy="0 0 0" xyz="0 0 0.055"/>
-      <xacro:base_color/>
-    </visual>
+      <mass value="5.0"/>
+      <inertia ixx="0.05" ixy="0" ixz="0" iyy="0.05" iyz="0" izz="0.05"/>
+    </inertial>
+    <visual>
+      <geometry><cylinder length="0.11" radius="0.26"/></geometry>
+      <origin rpy="0 0 0" xyz="0 0 0.055"/>
+      <material name="base_gray"/>
+    </visual>
+    <collision>
+      <geometry><cylinder length="0.11" radius="0.26"/></geometry>
+      <origin rpy="0 0 0" xyz="0 0 0.055"/>
+    </collision>
   </link>
   <joint name="base_to_pedestal_link" type="fixed">
     <parent link="base_link"/>
     <child link="pedestal_link"/>
-    <origin rpy="0 0 0"  xyz="0 0 0"/>
+    <origin rpy="0 0 0" xyz="0 0 0"/>
   </joint>
   <link name="pedestal_link">
-    <visual>
-      <geometry>
-        <cylinder length="0.94" radius="0.0254"/>
-      </geometry>
-      <origin rpy="0 0 0" xyz="0 0 0.58"/>
-      <xacro:base_color/>
-    </visual>
-  </link>
-  <link name="head_tilt_link">
-    <visual>
-      <geometry>
-        <mesh filename="package://inmoov_meshes/meshes/virtual.stl" scale="0.001 0.001 0.001"/>
-      </geometry>
-      <origin rpy="0 0 3.1415" xyz="0 0 0"/>
-      <xacro:frame_color/>
-    </visual>
-    <xacro:virtual_inertial/>
+    <inertial>
+      <origin rpy="0 0 0" xyz="0 0 0.47"/>
+      <mass value="2.0"/>
+      <inertia ixx="0.01" ixy="0" ixz="0" iyy="0.01" iyz="0" izz="0.01"/>
+    </inertial>
+    <visual>
+      <geometry><cylinder length="0.94" radius="0.0254"/></geometry>
+      <origin rpy="0 0 0" xyz="0 0 0.47"/>
+      <material name="base_gray"/>
+    </visual>
+    <collision>
+      <geometry><cylinder length="0.94" radius="0.0254"/></geometry>
+      <origin rpy="0 0 0" xyz="0 0 0.47"/>
+    </collision>
   </link>
   <joint name="pedestal_to_mid_stomach_joint" type="fixed">
     <parent link="pedestal_link"/>
     <child link="mid_stomach_link"/>
-     <origin rpy="0 0 0"  xyz="0 0 0"/>
-  </joint>
-  <xacro:torso covers="yes" />
+    <origin rpy="0 0 0" xyz="0 0 0.94"/>
+  </joint>
+  <link name="mid_stomach_link">
+    <inertial>
+      <origin rpy="0 0 0" xyz="0 0 0"/>
+      <mass value="1.0"/>
+      <inertia ixx="0.01" ixy="0" ixz="0" iyy="0.01" iyz="0" izz="0.01"/>
+    </inertial>
+    <visual>
+      <geometry><mesh filename="meshes/mid_stomach.stl" scale="0.001 0.001 0.001"/></geometry>
+      <origin rpy="0 0 0" xyz="0 0 0"/>
+      <material name="base_gray"/>
+    </visual>
+    <collision>
+      <geometry><mesh filename="meshes/mid_stomach.stl" scale="0.001 0.001 0.001"/></geometry>
+      <origin rpy="0 0 0" xyz="0 0 0"/>
+    </collision>
+  </link>
+  <joint name="mid_stomach_to_torso_joint" type="fixed">
+    <parent link="mid_stomach_link"/>
+    <child link="torso_link"/>
+    <origin rpy="0 0 0" xyz="0 0 0"/>
+  </joint>
+  <link name="torso_link">
+    <inertial>
+      <origin rpy="0 0 0" xyz="0 0 0"/>
+      <mass value="5.0"/>
+      <inertia ixx="0.1" ixy="0" ixz="0" iyy="0.1" iyz="0" izz="0.1"/>
+    </inertial>
+    <visual>
+      <geometry><mesh filename="meshes/torso.stl" scale="0.001 0.001 0.001"/></geometry>
+      <origin rpy="0 0 0" xyz="0 0 0"/>
+      <material name="base_gray"/>
+    </visual>
+    <collision>
+      <geometry><mesh filename="meshes/torso.stl" scale="0.001 0.001 0.001"/></geometry>
+      <origin rpy="0 0 0" xyz="0 0 0"/>
+    </collision>
+  </link>
+  <!-- Head stack (simplified but loadable in PyBullet). -->
+  <link name="head_tilt_link">
+    <inertial>
+      <origin rpy="0 0 0" xyz="0 0 0"/>
+      <mass value="0.2"/>
+      <inertia ixx="0.001" ixy="0" ixz="0" iyy="0.001" iyz="0" izz="0.001"/>
+    </inertial>
+    <visual>
+      <geometry><mesh filename="meshes/virtual.stl" scale="0.001 0.001 0.001"/></geometry>
+      <origin rpy="0 0 3.1415" xyz="0 0 0"/>
+      <material name="frame_green"/>
+    </visual>
+    <collision>
+      <geometry><mesh filename="meshes/virtual.stl" scale="0.001 0.001 0.001"/></geometry>
+      <origin rpy="0 0 3.1415" xyz="0 0 0"/>
+    </collision>
+  </link>
   <joint name="head_roll_joint" type="revolute">
-   <axis xyz="1 0 0"/>
-   <limit effort="1000.0" lower="${head_roll_joint_lower}" upper="${head_roll_joint_upper}" velocity="${head_roll_joint_velocity}" />
-   <origin rpy="0 0 3.1415" xyz="-0.0315  -0.001 0.4551"/>
-   <parent link="torso_link"/>
-   <child link="head_tilt_link"/>
-  </joint>
+    <parent link="torso_link"/>
+    <child link="head_tilt_link"/>
+    <origin rpy="0 0 3.1415" xyz="-0.0315 -0.001 0.4551"/>
+    <axis xyz="1 0 0"/>
+    <limit effort="1000.0" lower="-1.57" upper="1.57" velocity="2.0"/>
+  </joint>
+  <link name="head_base_link">
+    <inertial>
+      <origin rpy="0 0 0" xyz="0 0 0"/>
+      <mass value="1.0"/>
+      <inertia ixx="0.01" ixy="0" ixz="0" iyy="0.01" iyz="0" izz="0.01"/>
+    </inertial>
+    <visual>
+      <geometry><mesh filename="meshes/head_base.stl" scale="0.001 0.001 0.001"/></geometry>
+      <origin rpy="0 0 0" xyz="0 0 0"/>
+      <material name="base_gray"/>
+    </visual>
+    <collision>
+      <geometry><mesh filename="meshes/head_base.stl" scale="0.001 0.001 0.001"/></geometry>
+      <origin rpy="0 0 0" xyz="0 0 0"/>
+    </collision>
+  </link>
   <joint name="head_tilt_joint" type="revolute">
-   <axis xyz="0 1 0"/>
-   <limit effort="1000.0" lower="${head_tilt_joint_lower}" upper="${head_tilt_joint_upper}" velocity="${head_tilt_joint_velocity}" />
-   <origin rpy="0 0 3.1415" xyz="0 0 0"/>
-   <parent link="head_tilt_link"/>
-   <child link="head_base_link"/>
-  </joint>
-  <xacro:head covers="yes" />
-  <xacro:face covers="yes" />
+    <parent link="head_tilt_link"/>
+    <child link="head_base_link"/>
+    <origin rpy="0 0 3.1415" xyz="0 0 0"/>
+    <axis xyz="0 1 0"/>
+    <limit effort="1000.0" lower="-1.57" upper="1.57" velocity="2.0"/>
+  </joint>
+  <link name="skull_link">
+    <inertial>
+      <origin rpy="0 0 0" xyz="0 0 0"/>
+      <mass value="1.0"/>
+      <inertia ixx="0.01" ixy="0" ixz="0" iyy="0.01" iyz="0" izz="0.01"/>
+    </inertial>
+    <visual>
+      <geometry><mesh filename="meshes/skull.stl" scale="0.001 0.001 0.001"/></geometry>
+      <origin rpy="0 0 0" xyz="0 0 0"/>
+      <material name="base_gray"/>
+    </visual>
+    <collision>
+      <geometry><mesh filename="meshes/skull.stl" scale="0.001 0.001 0.001"/></geometry>
+      <origin rpy="0 0 0" xyz="0 0 0"/>
+    </collision>
+  </link>
+  <joint name="head_base_to_skull_joint" type="fixed">
+    <parent link="head_base_link"/>
+    <child link="skull_link"/>
+    <origin rpy="0 0 0" xyz="0 0 0"/>
+  </joint>
+  <link name="face_link">
+    <inertial>
+      <origin rpy="0 0 0" xyz="0 0 0"/>
+      <mass value="0.2"/>
+      <inertia ixx="0.001" ixy="0" ixz="0" iyy="0.001" iyz="0" izz="0.001"/>
+    </inertial>
+    <visual>
+      <geometry><mesh filename="meshes/face.stl" scale="0.001 0.001 0.001"/></geometry>
+      <origin rpy="0 0 0" xyz="0 0 0"/>
+      <material name="base_gray"/>
+    </visual>
+    <collision>
+      <geometry><mesh filename="meshes/face.stl" scale="0.001 0.001 0.001"/></geometry>
+      <origin rpy="0 0 0" xyz="0 0 0"/>
+    </collision>
+  </link>
   <joint name="face_joint" type="fixed">
-    <origin rpy="0 0 0" xyz="0.0637 0 0.079"/>
     <parent link="skull_link"/>
     <child link="face_link"/>
-  </joint>
-  <xacro:arm side="r" flip="1" covers="yes" />
+    <origin rpy="0 0 0" xyz="0.0637 0 0.079"/>
+  </joint>
+  <!-- Arms (high-level, loadable): shoulder base links are attached to torso; forearm->hand has wrist roll. -->
+  <link name="r_shoulder_base_link">
+    <visual>
+      <geometry><mesh filename="meshes/r_shoulder_base.stl" scale="0.001 0.001 0.001"/></geometry>
+      <origin rpy="0 0 0" xyz="0 0 0"/>
+      <material name="base_gray"/>
+    </visual>
+  </link>
   <joint name="r_shoulder_out_joint" type="revolute">
-   <axis xyz="1 0 0"/>
-   <limit effort="1000.0" lower="${r_shoulder_out_joint_lower}" upper="${r_shoulder_out_joint_upper}" velocity="${r_shoulder_out_joint_velocity}" />
-   <origin rpy="0 0 0" xyz="0 -0.143 0.298"/>
-   <parent link="torso_link"/>
-   <child link="r_shoulder_base_link"/>
-  </joint>
-  <xacro:hand side="r" flip="1" covers="yes" />
+    <parent link="torso_link"/>
+    <child link="r_shoulder_base_link"/>
+    <origin rpy="0 0 0" xyz="0 -0.143 0.298"/>
+    <axis xyz="1 0 0"/>
+    <limit effort="1000.0" lower="-2.0" upper="2.0" velocity="2.0"/>
+  </joint>
+  <link name="r_forearm_link">
+    <visual>
+      <geometry><mesh filename="meshes/r_forearm.stl" scale="0.001 0.001 0.001"/></geometry>
+      <origin rpy="0 0 0" xyz="0 0 0"/>
+      <material name="base_gray"/>
+    </visual>
+  </link>
+  <joint name="r_shoulderbase_to_r_forearm_joint" type="fixed">
+    <parent link="r_shoulder_base_link"/>
+    <child link="r_forearm_link"/>
+    <origin rpy="0 0 0" xyz="0 0 0"/>
+  </joint>
+  <link name="r_hand_link">
+    <visual>
+      <geometry><mesh filename="meshes/r_hand.stl" scale="0.001 0.001 0.001"/></geometry>
+      <origin rpy="0 0 0" xyz="0 0 0"/>
+      <material name="base_gray"/>
+    </visual>
+  </link>
   <joint name="r_wrist_roll_joint" type="revolute">
-   <axis xyz="0 0 1"/>
-   <limit effort="1000.0" lower="${r_wrist_roll_joint_lower}" upper="${r_wrist_roll_joint_upper}" velocity="${r_wrist_roll_joint_velocity}" />
-   <origin rpy="0 0 0" xyz="-0.0144 0.01  -0.2885"/>
-   <parent link="r_forearm_link"/>
-   <child link="r_hand_link"/>
-  </joint>
-  <xacro:arm side="l" flip="-1" covers="yes" />
+    <parent link="r_forearm_link"/>
+    <child link="r_hand_link"/>
+    <origin rpy="0 0 0" xyz="-0.0144 0.01 -0.2885"/>
+    <axis xyz="0 0 1"/>
+    <limit effort="1000.0" lower="-2.0" upper="2.0" velocity="4.0"/>
+  </joint>
+  <link name="l_shoulder_base_link">
+    <visual>
+      <geometry><mesh filename="meshes/l_shoulder_base.stl" scale="0.001 0.001 0.001"/></geometry>
+      <origin rpy="0 0 0" xyz="0 0 0"/>
+      <material name="base_gray"/>
+    </visual>
+  </link>
+  <!-- Left shoulder now has 3 sequential axes (yaw->pitch->roll) so we can animate X/Y/Z separately. -->
+  <link name="l_shoulder_yaw_link"/>
+  <joint name="l_shoulder_yaw_joint" type="revolute">
+    <parent link="torso_link"/>
+    <child link="l_shoulder_yaw_link"/>
+    <origin rpy="0 0 0" xyz="0 0.143 0.298"/>
+    <axis xyz="0 0 1"/>
+    <limit effort="1000.0" lower="-2.0" upper="2.0" velocity="2.0"/>
+  </joint>
+  <link name="l_shoulder_pitch_link"/>
+  <joint name="l_shoulder_pitch_joint" type="revolute">
+    <parent link="l_shoulder_yaw_link"/>
+    <child link="l_shoulder_pitch_link"/>
+    <origin rpy="0 0 0" xyz="0 0 0"/>
+    <axis xyz="0 1 0"/>
+    <limit effort="1000.0" lower="-2.0" upper="2.0" velocity="2.0"/>
+  </joint>
   <joint name="l_shoulder_out_joint" type="revolute">
-   <axis xyz="1 0 0"/>
-   <limit effort="1000.0" lower="${l_shoulder_out_joint_lower}" upper="${l_shoulder_out_joint_upper}" velocity="${l_shoulder_out_joint_velocity}" />
-   <origin rpy="0 0 0" xyz="0 0.143 0.298"/>
-   <parent link="torso_link"/>
-   <child link="l_shoulder_base_link"/>
-  </joint>
-  <xacro:hand side="l" flip="-1" covers="yes" />
+    <parent link="l_shoulder_pitch_link"/>
+    <child link="l_shoulder_base_link"/>
+    <origin rpy="0 0 0" xyz="0 0 0"/>
+    <axis xyz="1 0 0"/>
+    <limit effort="1000.0" lower="-2.0" upper="2.0" velocity="2.0"/>
+  </joint>
+  <link name="l_forearm_link">
+    <visual>
+      <geometry><mesh filename="meshes/l_forearm.stl" scale="0.001 0.001 0.001"/></geometry>
+      <origin rpy="0 0 0" xyz="0 0 0"/>
+      <material name="base_gray"/>
+    </visual>
+  </link>
+  <joint name="l_shoulderbase_to_l_forearm_joint" type="fixed">
+    <parent link="l_shoulder_base_link"/>
+    <child link="l_forearm_link"/>
+    <origin rpy="0 0 0" xyz="0 0 0"/>
+  </joint>
+  <link name="l_hand_link">
+    <visual>
+      <geometry><mesh filename="meshes/l_hand.stl" scale="0.001 0.001 0.001"/></geometry>
+      <origin rpy="0 0 0" xyz="0 0 0"/>
+      <material name="base_gray"/>
+    </visual>
+  </link>
   <joint name="l_wrist_roll_joint" type="revolute">
-   <axis xyz="0 0 1"/>
-   <limit effort="1000.0" lower="${l_wrist_roll_joint_lower}" upper="${l_wrist_roll_joint_upper}" velocity="${l_wrist_roll_joint_velocity}" />
-   <origin rpy="0 0 0" xyz="-0.0144 -0.01  -0.2885"/>
-   <parent link="l_forearm_link"/>
-   <child link="l_hand_link"/>
+    <parent link="l_forearm_link"/>
+    <child link="l_hand_link"/>
+    <origin rpy="0 0 0" xyz="-0.0144 -0.01 -0.2885"/>
+    <axis xyz="0 0 1"/>
+    <limit effort="1000.0" lower="-2.0" upper="2.0" velocity="4.0"/>
   </joint>
 </robot>
