Commit message: add of one more joint and neutralization of the rotz on the previous one
Everything should be working now, if any trouble persists, don't hesitate to send a text bro!

File: arm/left_arm.urdf (robot description, URDF)
Before this commit: robot left_arm_final, 27 links, 26 joints
Links:
- added link left_arm_rotz, mass 0.01
- added link left_shoulder_rotz_arm, mass 0.1
Joints:
- added joint jLeftArm_rotz: type revolute, parent left_upper_arm, child left_arm_rotz, origin xyz=-0.305 0 0 rpy=0 0 0, axis 0 0 -1, limit lower=-3.14 upper=3.14 effort=200 velocity=100.0
- added joint jLeftShoulder_rotz_arm: type revolute, parent left_shoulder_rotz_arm, child left_upper_arm, origin xyz=0 0 0 rpy=0 0 0, axis 0 0 -1, limit lower=-3.14 upper=3.14 effort=200 velocity=100.0
- joint jLeftElbow_roty: origin xyz=-0.305 0 0 rpy=0 0 0 -> xyz=0 0 0 rpy=0 0 0; parent left_upper_arm -> left_arm_rotz
- joint jLeftShoulder_roty: child left_upper_arm -> left_shoulder_rotz_arm
- joint jLeftShoulder_rotz: axis 0 0 -1 -> (none); limit lower=-3.14 upper=3.14 effort=200 velocity=100.0 -> (none); type revolute -> fixed
